Commit message: Add files via upload

File: test_robot_description/urdf/test_robot.xacro (robot description, xacro)
@@ -126,5 +126,5 @@
 <link name="servo_mount_v2_1">
   <inertial>
-    <origin xyz="0.022810444394987556 -1.5494500188104054e-09 -0.007692668094140112" rpy="0 0 0"/>
+    <origin xyz="0.022810444394987556 -1.5494500209788098e-09 -0.0026926680941401007" rpy="0 0 0"/>
     <mass value="0.28990445760104805"/>
     <inertia ixx="5.9e-05" iyy="0.00017" izz="0.000152" ixy="0.0" iyz="-0.0" ixz="6e-06"/>
@@ -146,10 +146,10 @@
 <link name="camera_mount_v2_1">
   <inertial>
-    <origin xyz="0.009999999999998233 2.0903417885520525e-16 0.0030000000000000443" rpy="0 0 0"/>
+    <origin xyz="0.009999999999998233 2.0686577451023425e-16 0.0030000000000000304" rpy="0 0 0"/>
     <mass value="0.012966923677691866"/>
     <inertia ixx="5e-06" iyy="5e-06" izz="1e-05" ixy="0.0" iyz="-0.0" ixz="-0.0"/>
   </inertial>
   <visual>
-    <origin xyz="-0.19055 -0.0025 -0.07723" rpy="0 0 0"/>
+    <origin xyz="-0.19055 -0.0025 -0.08223" rpy="0 0 0"/>
     <geometry>
       <mesh filename="package://test_robot_description/meshes/camera_mount_v2_1.stl" scale="0.001 0.001 0.001"/>
@@ -158,5 +158,5 @@
   </visual>
   <collision>
-    <origin xyz="-0.19055 -0.0025 -0.07723" rpy="0 0 0"/>
+    <origin xyz="-0.19055 -0.0025 -0.08223" rpy="0 0 0"/>
     <geometry>
       <mesh filename="package://test_robot_description/meshes/camera_mount_v2_1.stl" scale="0.001 0.001 0.001"/>
@@ -166,10 +166,10 @@
 <link name="camera_v4_1">
   <inertial>
-    <origin xyz="0.05512009244754448 3.3471489468972493e-15 0.045945900256365614" rpy="0 0 0"/>
+    <origin xyz="0.003870092447544521 3.342378457338313e-15 0.022445900256365642" rpy="0 0 0"/>
     <mass value="0.6054290756769216"/>
     <inertia ixx="0.000158" iyy="0.000199" izz="0.000199" ixy="-0.0" iyz="0.0" ixz="-0.0"/>
   </inertial>
   <visual>
-    <origin xyz="-0.1599 -0.0025 -0.05718" rpy="0 0 0"/>
+    <origin xyz="-0.21055 -0.0025 -0.08623" rpy="0 0 0"/>
     <geometry>
       <mesh filename="package://test_robot_description/meshes/camera_v4_1.stl" scale="0.001 0.001 0.001"/>
@@ -178,5 +178,5 @@
   </visual>
   <collision>
-    <origin xyz="-0.1599 -0.0025 -0.05718" rpy="0 0 0"/>
+    <origin xyz="-0.21055 -0.0025 -0.08623" rpy="0 0 0"/>
     <geometry>
       <mesh filename="package://test_robot_description/meshes/camera_v4_1.stl" scale="0.001 0.001 0.001"/>
@@ -217,12 +217,12 @@
 </joint>
 <joint name="Revolute 7" type="continuous">
-  <origin xyz="0.03815 0.0 0.01755" rpy="0 0 0"/>
+  <origin xyz="0.03815 0.0 0.02255" rpy="0 0 0"/>
   <parent link="servo_mount_v2_1"/>
   <child link="camera_mount_v2_1"/>
   <axis xyz="0.0 -0.0 1.0"/>
 </joint>
-<joint name="Rigid 8" type="fixed">
-  <origin xyz="0.0075 0.0 -0.0025" rpy="0 0 0"/>
-  <parent link="servo_mount_v2_1"/>
+<joint name="Rigid 9" type="fixed">
+  <origin xyz="0.02 0.0 0.004" rpy="0 0 0"/>
+  <parent link="camera_mount_v2_1"/>
   <child link="camera_v4_1"/>
 </joint>

Commit message: Add files via upload

File: test_robot_description/urdf/test_robot.xacro (robot description, xacro)
@@ -84,5 +84,5 @@
   </collision>
 </link>
-<link name="castor_v1_1">
+<link name="right_castor_1">
   <inertial>
     <origin xyz="-0.015000000000078367 0.019999999999999976 -0.025454061421393216" rpy="0 0 0"/>
@@ -93,5 +93,5 @@
     <origin xyz="-0.1474 0.1449 -0.05468" rpy="0 0 0"/>
     <geometry>
-      <mesh filename="package://test_robot_description/meshes/castor_v1_1.stl" scale="0.001 0.001 0.001"/>
+      <mesh filename="package://test_robot_description/meshes/right_castor_1.stl" scale="0.001 0.001 0.001"/>
     </geometry>
     <material name="aluminum_satin"/>
@@ -100,9 +100,9 @@
     <origin xyz="-0.1474 0.1449 -0.05468" rpy="0 0 0"/>
     <geometry>
-      <mesh filename="package://test_robot_description/meshes/castor_v1_1.stl" scale="0.001 0.001 0.001"/>
-    </geometry>
-  </collision>
-</link>
-<link name="ydlidar_x4_v1_1">
+      <mesh filename="package://test_robot_description/meshes/right_castor_1.stl" scale="0.001 0.001 0.001"/>
+    </geometry>
+  </collision>
+</link>
+<link name="ydlidar_x4_1">
   <inertial>
     <origin xyz="0.008294099570319522 -3.8163916471489756e-17 0.034201142222791026" rpy="0 0 0"/>
@@ -113,5 +113,5 @@
     <origin xyz="-0.0 -0.0025 -0.11668" rpy="0 0 0"/>
     <geometry>
-      <mesh filename="package://test_robot_description/meshes/ydlidar_x4_v1_1.stl" scale="0.001 0.001 0.001"/>
+      <mesh filename="package://test_robot_description/meshes/ydlidar_x4_1.stl" scale="0.001 0.001 0.001"/>
     </geometry>
     <material name="steel_satin"/>
@@ -120,9 +120,9 @@
     <origin xyz="-0.0 -0.0025 -0.11668" rpy="0 0 0"/>
     <geometry>
-      <mesh filename="package://test_robot_description/meshes/ydlidar_x4_v1_1.stl" scale="0.001 0.001 0.001"/>
-    </geometry>
-  </collision>
-</link>
-<link name="servo_mount_v2_1">
+      <mesh filename="package://test_robot_description/meshes/ydlidar_x4_1.stl" scale="0.001 0.001 0.001"/>
+    </geometry>
+  </collision>
+</link>
+<link name="servo_mount_1">
   <inertial>
     <origin xyz="0.022810444394987556 -1.5494500209788098e-09 -0.0026926680941401007" rpy="0 0 0"/>
@@ -133,5 +133,5 @@
     <origin xyz="-0.1524 -0.0025 -0.05968" rpy="0 0 0"/>
     <geometry>
-      <mesh filename="package://test_robot_description/meshes/servo_mount_v2_1.stl" scale="0.001 0.001 0.001"/>
+      <mesh filename="package://test_robot_description/meshes/servo_mount_1.stl" scale="0.001 0.001 0.001"/>
     </geometry>
     <material name="acrylic_clear"/>
@@ -140,9 +140,9 @@
     <origin xyz="-0.1524 -0.0025 -0.05968" rpy="0 0 0"/>
     <geometry>
-      <mesh filename="package://test_robot_description/meshes/servo_mount_v2_1.stl" scale="0.001 0.001 0.001"/>
-    </geometry>
-  </collision>
-</link>
-<link name="camera_mount_v2_1">
+      <mesh filename="package://test_robot_description/meshes/servo_mount_1.stl" scale="0.001 0.001 0.001"/>
+    </geometry>
+  </collision>
+</link>
+<link name="camera_mount_1">
   <inertial>
     <origin xyz="0.009999999999998233 2.0686577451023425e-16 0.0030000000000000304" rpy="0 0 0"/>
@@ -153,5 +153,5 @@
     <origin xyz="-0.19055 -0.0025 -0.08223" rpy="0 0 0"/>
     <geometry>
-      <mesh filename="package://test_robot_description/meshes/camera_mount_v2_1.stl" scale="0.001 0.001 0.001"/>
+      <mesh filename="package://test_robot_description/meshes/camera_mount_1.stl" scale="0.001 0.001 0.001"/>
     </geometry>
     <material name="paek_beige"/>
@@ -160,9 +160,9 @@
     <origin xyz="-0.19055 -0.0025 -0.08223" rpy="0 0 0"/>
     <geometry>
-      <mesh filename="package://test_robot_description/meshes/camera_mount_v2_1.stl" scale="0.001 0.001 0.001"/>
-    </geometry>
-  </collision>
-</link>
-<link name="camera_v4_1">
+      <mesh filename="package://test_robot_description/meshes/camera_mount_1.stl" scale="0.001 0.001 0.001"/>
+    </geometry>
+  </collision>
+</link>
+<link name="camera_1">
   <inertial>
     <origin xyz="0.003870092447544521 3.342378457338313e-15 0.022445900256365642" rpy="0 0 0"/>
@@ -173,5 +173,5 @@
     <origin xyz="-0.21055 -0.0025 -0.08623" rpy="0 0 0"/>
     <geometry>
-      <mesh filename="package://test_robot_description/meshes/camera_v4_1.stl" scale="0.001 0.001 0.001"/>
+      <mesh filename="package://test_robot_description/meshes/camera_1.stl" scale="0.001 0.001 0.001"/>
     </geometry>
     <material name="steel_satin"/>
@@ -180,9 +180,9 @@
     <origin xyz="-0.21055 -0.0025 -0.08623" rpy="0 0 0"/>
     <geometry>
-      <mesh filename="package://test_robot_description/meshes/camera_v4_1.stl" scale="0.001 0.001 0.001"/>
-    </geometry>
-  </collision>
-</link>
-<joint name="Revolute 1" type="continuous">
+      <mesh filename="package://test_robot_description/meshes/camera_1.stl" scale="0.001 0.001 0.001"/>
+    </geometry>
+  </collision>
+</link>
+<joint name="right_drive" type="continuous">
   <origin xyz="-0.116382 -0.183454 0.035" rpy="0 0 0"/>
   <parent link="base_link"/>
@@ -190,5 +190,5 @@
   <axis xyz="0.0 -1.0 -0.0"/>
 </joint>
-<joint name="Revolute 2" type="continuous">
+<joint name="left_drive" type="continuous">
   <origin xyz="-0.116418 0.188454 0.035" rpy="0 0 0"/>
   <parent link="base_link"/>
@@ -204,26 +204,26 @@
   <origin xyz="0.1474 -0.1449 0.05468" rpy="0 0 0"/>
   <parent link="base_link"/>
-  <child link="castor_v1_1"/>
+  <child link="right_castor_1"/>
 </joint>
 <joint name="Rigid 5" type="fixed">
   <origin xyz="0.0 0.0025 0.11668" rpy="0 0 0"/>
   <parent link="base_link"/>
-  <child link="ydlidar_x4_v1_1"/>
+  <child link="ydlidar_x4_1"/>
 </joint>
 <joint name="Rigid 6" type="fixed">
   <origin xyz="0.1524 0.0025 0.05968" rpy="0 0 0"/>
   <parent link="base_link"/>
-  <child link="servo_mount_v2_1"/>
-</joint>
-<joint name="Revolute 7" type="continuous">
+  <child link="servo_mount_1"/>
+</joint>
+<joint name="camera_joint" type="continuous">
   <origin xyz="0.03815 0.0 0.02255" rpy="0 0 0"/>
-  <parent link="servo_mount_v2_1"/>
-  <child link="camera_mount_v2_1"/>
+  <parent link="servo_mount_1"/>
+  <child link="camera_mount_1"/>
   <axis xyz="0.0 -0.0 1.0"/>
 </joint>
 <joint name="Rigid 9" type="fixed">
   <origin xyz="0.02 0.0 0.004" rpy="0 0 0"/>
-  <parent link="camera_mount_v2_1"/>
-  <child link="camera_v4_1"/>
+  <parent link="camera_mount_1"/>
+  <child link="camera_1"/>
 </joint>
 </robot>

Commit message: Add files via upload

File: test_robot_description/urdf/test_robot.xacro (robot description, xacro)
@@ -24,5 +24,5 @@
   </collision>
 </link>
-<link name="right_wheel_1">
+<link name="right_wheel">
   <inertial>
     <origin xyz="-3.4200742424217445e-07 -0.0073158880868150755 -4.197731875474342e-06" rpy="0 0 0"/>
@@ -44,5 +44,5 @@
   </collision>
 </link>
-<link name="left_wheel_1">
+<link name="left_wheel">
   <inertial>
     <origin xyz="3.4200744483681156e-07 0.007315888086814659 3.864337692033315e-06" rpy="0 0 0"/>
@@ -64,5 +64,5 @@
   </collision>
 </link>
-<link name="left_castor_1">
+<link name="left_castor">
   <inertial>
     <origin xyz="-0.015000000000078645 -0.01999999999999974 -0.025454061421393108" rpy="0 0 0"/>
@@ -84,5 +84,5 @@
   </collision>
 </link>
-<link name="right_castor_1">
+<link name="right_castor">
   <inertial>
     <origin xyz="-0.015000000000078367 0.019999999999999976 -0.025454061421393216" rpy="0 0 0"/>
@@ -104,5 +104,5 @@
   </collision>
 </link>
-<link name="ydlidar_x4_1">
+<link name="ydlidar_x4">
   <inertial>
     <origin xyz="0.008294099570319522 -3.8163916471489756e-17 0.034201142222791026" rpy="0 0 0"/>
@@ -111,18 +111,18 @@
   </inertial>
   <visual>
+    <origin xyz="-0.0 -0.0025 -0.16668" rpy="0 0 0"/>
+    <geometry>
+      <mesh filename="package://test_robot_description/meshes/ydlidar_x4_1.stl" scale="0.001 0.001 0.001"/>
+    </geometry>
+    <material name="steel_satin"/>
+  </visual>
+  <collision>
     <origin xyz="-0.0 -0.0025 -0.11668" rpy="0 0 0"/>
     <geometry>
       <mesh filename="package://test_robot_description/meshes/ydlidar_x4_1.stl" scale="0.001 0.001 0.001"/>
     </geometry>
-    <material name="steel_satin"/>
-  </visual>
-  <collision>
-    <origin xyz="-0.0 -0.0025 -0.11668" rpy="0 0 0"/>
-    <geometry>
-      <mesh filename="package://test_robot_description/meshes/ydlidar_x4_1.stl" scale="0.001 0.001 0.001"/>
-    </geometry>
-  </collision>
-</link>
-<link name="servo_mount_1">
+  </collision>
+</link>
+<link name="servo_mount">
   <inertial>
     <origin xyz="0.022810444394987556 -1.5494500209788098e-09 -0.0026926680941401007" rpy="0 0 0"/>
@@ -144,5 +144,5 @@
   </collision>
 </link>
-<link name="camera_mount_1">
+<link name="camera_mount">
   <inertial>
     <origin xyz="0.009999999999998233 2.0686577451023425e-16 0.0030000000000000304" rpy="0 0 0"/>
@@ -164,5 +164,5 @@
   </collision>
 </link>
-<link name="camera_1">
+<link name="camera">
   <inertial>
     <origin xyz="0.003870092447544521 3.342378457338313e-15 0.022445900256365642" rpy="0 0 0"/>
@@ -187,11 +187,11 @@
   <origin xyz="-0.116382 -0.183454 0.035" rpy="0 0 0"/>
   <parent link="base_link"/>
-  <child link="right_wheel_1"/>
-  <axis xyz="0.0 -1.0 -0.0"/>
+  <child link="right_wheel"/>
+  <axis xyz="0.0 1.0 -0.0"/>
 </joint>
 <joint name="left_drive" type="continuous">
   <origin xyz="-0.116418 0.188454 0.035" rpy="0 0 0"/>
   <parent link="base_link"/>
-  <child link="left_wheel_1"/>
+  <child link="left_wheel"/>
   <axis xyz="-0.0 1.0 0.0"/>
 </joint>
@@ -199,31 +199,31 @@
   <origin xyz="0.1474 0.1499 0.05468" rpy="0 0 0"/>
   <parent link="base_link"/>
-  <child link="left_castor_1"/>
+  <child link="left_castor"/>
 </joint>
 <joint name="Rigid 4" type="fixed">
   <origin xyz="0.1474 -0.1449 0.05468" rpy="0 0 0"/>
   <parent link="base_link"/>
-  <child link="right_castor_1"/>
+  <child link="right_castor"/>
 </joint>
 <joint name="Rigid 5" type="fixed">
-  <origin xyz="0.0 0.0025 0.11668" rpy="0 0 0"/>
-  <parent link="base_link"/>
-  <child link="ydlidar_x4_1"/>
+  <origin xyz="0.0 0.025 0.16668" rpy="0 0 0"/>
+  <parent link="base_link"/>
+  <child link="ydlidar_x4"/>
 </joint>
 <joint name="Rigid 6" type="fixed">
   <origin xyz="0.1524 0.0025 0.05968" rpy="0 0 0"/>
   <parent link="base_link"/>
-  <child link="servo_mount_1"/>
+  <child link="servo_mount"/>
 </joint>
 <joint name="camera_joint" type="continuous">
   <origin xyz="0.03815 0.0 0.02255" rpy="0 0 0"/>
-  <parent link="servo_mount_1"/>
-  <child link="camera_mount_1"/>
+  <parent link="servo_mount"/>
+  <child link="camera_mount"/>
   <axis xyz="0.0 -0.0 1.0"/>
 </joint>
 <joint name="Rigid 9" type="fixed">
   <origin xyz="0.02 0.0 0.004" rpy="0 0 0"/>
-  <parent link="camera_mount_1"/>
-  <child link="camera_1"/>
+  <parent link="camera_mount"/>
+  <child link="camera"/>
 </joint>
 </robot>

Commit message: Add files via upload

File: test_robot_description/urdf/test_robot.xacro (robot description, xacro)
@@ -184,4 +184,84 @@
   </collision>
 </link>
+<link name="MPU_6050">
+  <inertial>
+    <origin xyz="-3.1355336134285696e-05 -0.050012226392699075 0.0009153763215413793" rpy="0 0 0"/>
+    <mass value="0.004148060593361584"/>
+    <inertia ixx="0.0" iyy="0.0" izz="0.0" ixy="-0.0" iyz="-0.0" ixz="0.0"/>
+  </inertial>
+  <visual>
+    <origin xyz="0.0 -0.1549 -0.05968" rpy="0 0 0"/>
+    <geometry>
+      <mesh filename="package://test_robot_description/meshes/MPU_6050_1.stl" scale="0.001 0.001 0.001"/>
+    </geometry>
+    <material name="steel_satin"/>
+  </visual>
+  <collision>
+    <origin xyz="0.0 -0.1549 -0.05968" rpy="0 0 0"/>
+    <geometry>
+      <mesh filename="package://test_robot_description/meshes/MPU_6050_1.stl" scale="0.001 0.001 0.001"/>
+    </geometry>
+  </collision>
+</link>
+<link name="ADXL335">
+  <inertial>
+    <origin xyz="4.6126231438677886e-05 -0.025102857569161613 0.0004384677831028097" rpy="0 0 0"/>
+    <mass value="0.0022661803844448835"/>
+    <inertia ixx="0.0" iyy="0.0" izz="0.0" ixy="0.0" iyz="0.0" ixz="-0.0"/>
+  </inertial>
+  <visual>
+    <origin xyz="0.0 -0.1549 -0.05968" rpy="0 0 0"/>
+    <geometry>
+      <mesh filename="package://test_robot_description/meshes/ADXL335_1.stl" scale="0.001 0.001 0.001"/>
+    </geometry>
+    <material name="opaque202209238"/>
+  </visual>
+  <collision>
+    <origin xyz="0.0 -0.1549 -0.05968" rpy="0 0 0"/>
+    <geometry>
+      <mesh filename="package://test_robot_description/meshes/ADXL335_1.stl" scale="0.001 0.001 0.001"/>
+    </geometry>
+  </collision>
+</link>
+<link name="MPU_9250">
+  <inertial>
+    <origin xyz="-4.0745935269562253e-05 0.049982746308101816 0.0010543416597268984" rpy="0 0 0"/>
+    <mass value="0.006431034767624054"/>
+    <inertia ixx="0.0" iyy="0.0" izz="0.0" ixy="-0.0" iyz="-0.0" ixz="0.0"/>
+  </inertial>
+  <visual>
+    <origin xyz="-0.0 0.1499 -0.05968" rpy="0 0 0"/>
+    <geometry>
+      <mesh filename="package://test_robot_description/meshes/MPU_9250_1.stl" scale="0.001 0.001 0.001"/>
+    </geometry>
+    <material name="silver_default"/>
+  </visual>
+  <collision>
+    <origin xyz="-0.0 0.1499 -0.05968" rpy="0 0 0"/>
+    <geometry>
+      <mesh filename="package://test_robot_description/meshes/MPU_9250_1.stl" scale="0.001 0.001 0.001"/>
+    </geometry>
+  </collision>
+</link>
+<link name="QMC5883">
+  <inertial>
+    <origin xyz="3.957074476157516e-05 0.02470495460938099 0.0007776122652584164" rpy="0 0 0"/>
+    <mass value="0.0022004092587126446"/>
+    <inertia ixx="0.0" iyy="0.0" izz="0.0" ixy="0.0" iyz="0.0" ixz="-0.0"/>
+  </inertial>
+  <visual>
+    <origin xyz="-0.0 0.1499 -0.05968" rpy="0 0 0"/>
+    <geometry>
+      <mesh filename="package://test_robot_description/meshes/QMC5883_1.stl" scale="0.001 0.001 0.001"/>
+    </geometry>
+    <material name="steel_satin"/>
+  </visual>
+  <collision>
+    <origin xyz="-0.0 0.1499 -0.05968" rpy="0 0 0"/>
+    <geometry>
+      <mesh filename="package://test_robot_description/meshes/QMC5883_1.stl" scale="0.001 0.001 0.001"/>
+    </geometry>
+  </collision>
+</link>
 <joint name="right_drive" type="continuous">
   <origin xyz="-0.116382 -0.183454 0.035" rpy="0 0 0"/>
@@ -207,5 +287,5 @@
 </joint>
 <joint name="Rigid 5" type="fixed">
-  <origin xyz="0.0 0.025 0.16668" rpy="0 0 0"/>
+  <origin xyz="0.0 0.0025 0.16668" rpy="0 0 0"/>
   <parent link="base_link"/>
   <child link="ydlidar_x4"/>
@@ -227,3 +307,23 @@
   <child link="camera"/>
 </joint>
+<joint name="Rigid 10" type="fixed">
+  <origin xyz="0.0 0.1549 0.05968" rpy="0 0 0"/>
+  <parent link="base_link"/>
+  <child link="MPU_6050"/>
+</joint>
+<joint name="Rigid 11" type="fixed">
+  <origin xyz="0.0 0.1549 0.05968" rpy="0 0 0"/>
+  <parent link="base_link"/>
+  <child link="ADXL335"/>
+</joint>
+<joint name="Rigid 12" type="fixed">
+  <origin xyz="0.0 -0.1499 0.05968" rpy="0 0 0"/>
+  <parent link="base_link"/>
+  <child link="MPU_9250"/>
+</joint>
+<joint name="Rigid 13" type="fixed">
+  <origin xyz="0.0 -0.1499 0.05968" rpy="0 0 0"/>
+  <parent link="base_link"/>
+  <child link="QMC5883"/>
+</joint>
 </robot>

Commit message: Add files via upload

File: test_robot_description/urdf/test_robot.xacro (robot description, xacro)
@@ -215,5 +215,5 @@
       <mesh filename="package://test_robot_description/meshes/ADXL335_1.stl" scale="0.001 0.001 0.001"/>
     </geometry>
-    <material name="opaque202209238"/>
+    <material name="steel_satin"/>
   </visual>
   <collision>
@@ -235,5 +235,5 @@
       <mesh filename="package://test_robot_description/meshes/MPU_9250_1.stl" scale="0.001 0.001 0.001"/>
     </geometry>
-    <material name="silver_default"/>
+    <material name="steel_satin"/>
   </visual>
   <collision>
